File: KiCad/jam-pad/jam-pad_plate.kicad_pcb (KiCad board)
At the start: 2 copper layers, 137.6 x 71.4 mm, 5 parts

Commit message: routing adjustments, ec11 standoff, need to fix drc kms
Parts:
- added REF**: MountingHole_2.2mm_M2_Pad, MountingHole:MountingHole_2.2mm_M2_Pad, F.Cu at (60.3, 38.5)
- added REF**: MountingHole_2.2mm_M2_Pad, MountingHole:MountingHole_2.2mm_M2_Pad, F.Cu at (60.3, 69.8)
- added SW14: RotaryEncoder_Switch, Keebio-Parts:RotaryEncoder_Alps_EC11E-Switch_Vertical_H20mm, F.Cu at (60.3, 54.0)
Other:
- board size 137.6 x 71.4 mm -> 137.3 x 71.4 mm
Changed lines of the file:
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@@
   (net 0 "")
   (footprint "MountingHole:MountingHole_2.2mm_M2_Pad" (layer "F.Cu")
+    (at 60.325 38.496875)
+    (descr "Mounting Hole 2.2mm, M2")
+    (tags "mounting hole 2.2mm m2")
+    (attr exclude_from_pos_files exclude_from_bom)
+    (fp_text reference "REF**" (at 0 -3.2) (layer "F.SilkS") hide
+        (effects (font (size 1 1) (thickness 0.15)))
+    )
+    (fp_text value "MountingHole_2.2mm_M2_Pad" (at 0 3.2) (layer "F.Fab") hide
+        (effects (font (size 1 1) (thickness 0.15)))
+    )
+    (fp_text user "${REFERENCE}" (at 0 0) (layer "F.Fab")
+        (effects (font (size 1 1) (thickness 0.15)))
+    )
+    (fp_circle (center 0 0) (end 2.2 0)
+      (stroke (width 0.15) (type solid)) (fill none) (layer "Cmts.User"))
+    (fp_circle (center 0 0) (end 2.45 0)
+      (stroke (width 0.05) (type solid)) (fill none) (layer "F.CrtYd"))
+    (pad "1" thru_hole circle (at 0 0) (size 4.4 4.4) (drill 2.2) (layers "*.Cu" "*.Mask"))
+  )
+  (footprint "MountingHole:MountingHole_2.2mm_M2_Pad" (layer "F.Cu")
     (at 31.353125 53.975001 90)
     (descr "Mounting Hole 2.2mm, M2")
@@
       (stroke (width 0.05) (type solid)) (fill none) (layer "F.CrtYd"))
     (pad "1" thru_hole circle (at 0 0 180) (size 4.4 4.4) (drill 2.2) (layers "*.Cu" "*.Mask"))
+  )
+  (footprint "Keebio-Parts:RotaryEncoder_Alps_EC11E-Switch_Vertical_H20mm" (layer "F.Cu")
+    (at 60.325 53.975 90)
+    (descr "Alps rotary encoder, EC12E... with switch, vertical shaft, http://www.alps.com/prod/info/E/HTML/Encoder/Incremental/EC11/EC11E15204A3.html")
+    (tags "rotary encoder")
+    (property "Sheetfile" "jam-pad.kicad_sch")
+    (property "Sheetname" "")
+    (property "ki_description" "Rotary encoder, dual channel, incremental quadrate outputs, with switch")
+    (property "ki_keywords" "rotary switch encoder switch push button")
+    (attr through_hole)
+    (fp_text reference "SW14" (at -4.7 -7.2 90) (layer "F.SilkS")
+        (effects (font (size 1 1) (thickness 0.15)))
+    )
+    (fp_text value "RotaryEncoder_Switch" (at 0 7.9 90) (layer "F.Fab")
+        (effects (font (size 1 1) (thickness 0.15)))
+    )
+    (fp_text user "${REFERENCE}" (at 3.6 3.8 90) (layer "F.Fab")
+        (effects (font (size 1 1) (thickness 0.15)))
+    )
+    (fp_line (start -7.8 -4.1) (end -7.2 -4.1)
+      (stroke (width 0.12) (type solid)) (layer "F.SilkS"))
+    (fp_line (start -7.5 -3.8) (end -7.8 -4.1)
+      (stroke (width 0.12) (type solid)) (layer "F.SilkS"))
+    (fp_line (start -7.2 -4.1) (end -7.5 -3.8)
+      (stroke (width 0.12) (type solid)) (layer "F.SilkS"))
+    (fp_line (start -6.1 -5.9) (end -6.1 5.9)
+      (stroke (width 0.12) (type solid)) (layer "F.SilkS"))
+    (fp_line (start -2 -5.9) (end -6.1 -5.9)
+      (stroke (width 0.12) (type solid)) (layer "F.SilkS"))
+    (fp_line (start -2 5.9) (end -6.1 5.9)
+      (stroke (width 0.12) (type solid)) (layer "F.SilkS"))
+    (fp_line (start -0.5 0) (end 0.5 0)
+      (stroke (width 0.12) (type solid)) (layer "F.SilkS"))
+    (fp_line (start 0 -0.5) (end 0 0.5)
+      (stroke (width 0.12) (type solid)) (layer "F.SilkS"))
+    (fp_line (start 2 -5.9) (end 6.1 -5.9)
+      (stroke (width 0.12) (type solid)) (layer "F.SilkS"))
+    (fp_line (start 6.1 -5.9) (end 6.1 -3.5)
+      (stroke (width 0.12) (type solid)) (layer "F.SilkS"))
+    (fp_line (start 6.1 -1.3) (end 6.1 1.3)
+      (stroke (width 0.12) (type solid)) (layer "F.SilkS"))
+    (fp_line (start 6.1 3.5) (end 6.1 5.9)
+      (stroke (width 0.12) (type solid)) (layer "F.SilkS"))
+    (fp_line (start 6.1 5.9) (end 2 5.9)
+      (stroke (width 0.12) (type solid)) (layer "F.SilkS"))
+    (fp_circle (center 0 0) (end 3 0)
+      (stroke (width 0.12) (type solid)) (fill none) (layer "F.SilkS"))
+    (fp_line (start -9 -7.1) (end -9 7.1)
+      (stroke (width 0.05) (type solid)) (layer "F.CrtYd"))
+    (fp_line (start -9 -7.1) (end 8.5 -7.1)
+      (stroke (width 0.05) (type solid)) (layer "F.CrtYd"))
+    (fp_line (start 8.5 7.1) (end -9 7.1)
+      (stroke (width 0.05) (type solid)) (layer "F.CrtYd"))
+    (fp_line (start 8.5 7.1) (end 8.5 -7.1)
+      (stroke (width 0.05) (type solid)) (layer "F.CrtYd"))
+    (fp_line (start -6 -4.7) (end -5 -5.8)
+      (stroke (width 0.12) (type solid)) (layer "F.Fab"))
+    (fp_line (start -6 5.8) (end -6 -4.7)
+      (stroke (width 0.12) (type solid)) (layer "F.Fab"))
+    (fp_line (start -5 -5.8) (end 6 -5.8)
+      (stroke (width 0.12) (type solid)) (layer "F.Fab"))
+    (fp_line (start -3 0) (end 3 0)
+      (stroke (width 0.12) (type solid)) (layer "F.Fab"))
+    (fp_line (start 0 -3) (end 0 3)
+      (stroke (width 0.12) (type solid)) (layer "F.Fab"))
+    (fp_line (start 6 -5.8) (end 6 5.8)
+      (stroke (width 0.12) (type solid)) (layer "F.Fab"))
+    (fp_line (start 6 5.8) (end -6 5.8)
+      (stroke (width 0.12) (type solid)) (layer "F.Fab"))
+    (fp_circle (center 0 0) (end 3 0)
+      (stroke (width 0.12) (type solid)) (fill none) (layer "F.Fab"))
+    (pad "A" thru_hole rect (at -7.5 -2.5 90) (size 2 2) (drill 1) (layers "*.Cu" "*.Mask")
+      (pinfunction "A") (pintype "passive"))
+    (pad "B" thru_hole circle (at -7.5 2.5 90) (size 2 2) (drill 1) (layers "*.Cu" "*.Mask")
+      (pinfunction "B") (pintype "passive"))
+    (pad "C" thru_hole circle (at -7.5 0 90) (size 2 2) (drill 1) (layers "*.Cu" "*.Mask")
+      (pinfunction "C") (pintype "passive"))
+    (pad "MP" thru_hole rect (at 0 -5.6 90) (size 3.2 2) (drill oval 2.8 1.5) (layers "*.Cu" "*.Mask"))
+    (pad "MP" thru_hole rect (at 0 5.6 90) (size 3.2 2) (drill oval 2.8 1.5) (layers "*.Cu" "*.Mask"))
+    (pad "S1" thru_hole circle (at 7 2.5 90) (size 2 2) (drill 1) (layers "*.Cu" "*.Mask")
+      (pinfunction "S1") (pintype "passive"))
+    (pad "S2" thru_hole circle (at 7 -2.5 90) (size 2 2) (drill 1) (layers "*.Cu" "*.Mask")
+      (pinfunction "S2") (pintype "passive"))
+    (model "${KICAD6_3DMODEL_DIR}/Rotary_Encoder.3dshapes/RotaryEncoder_Alps_EC11E-Switch_Vertical_H20mm.wrl"
+      (offset (xyz 0 0 0))
+      (scale (xyz 1 1 1))
+      (rotate (xyz 0 0 0))
+    )
+  )
+  (footprint "MountingHole:MountingHole_2.2mm_M2_Pad" (layer "F.Cu")
+    (at 60.325 69.85)
+    (descr "Mounting Hole 2.2mm, M2")
+    (tags "mounting hole 2.2mm m2")
+    (attr exclude_from_pos_files exclude_from_bom)
+    (fp_text reference "REF**" (at 0 -3.2) (layer "F.SilkS") hide
+        (effects (font (size 1 1) (thickness 0.15)))
+    )
+    (fp_text value "MountingHole_2.2mm_M2_Pad" (at 0 3.2) (layer "F.Fab") hide
+        (effects (font (size 1 1) (thickness 0.15)))
+    )
+    (fp_text user "${REFERENCE}" (at 0 0) (layer "F.Fab")
+        (effects (font (size 1 1) (thickness 0.15)))
+    )
+    (fp_circle (center 0 0) (end 2.2 0)
+      (stroke (width 0.15) (type solid)) (fill none) (layer "Cmts.User"))
+    (fp_circle (center 0 0) (end 2.45 0)
+      (stroke (width 0.05) (type solid)) (fill none) (layer "F.CrtYd"))
+    (pad "1" thru_hole circle (at 0 0) (size 4.4 4.4) (drill 2.2) (layers "*.Cu" "*.Mask"))
   )
   (gr_circle (center 60.325 53.975) (end 61.11875 25.4)
@@
   (gr_arc (start 32.54375 47.241902) (mid 42.655347 31.514313) (end 60.325 25.4)
     (stroke (width 0.1) (type default)) (layer "Edge.Cuts"))
-  (gr_line (start 157.956267 48.41875) (end 161.798 48.41875)
+  (gr_line (start 157.956267 48.41875) (end 161.528325 48.41875)
     (stroke (width 0.1) (type solid)) (layer "Edge.Cuts"))
   (gr_arc (start 133.99375 60.975) (mid 133.640197 60.828553) (end 133.49375 60.475)
@@
   (gr_line (start 95.89375 66.025) (end 108.89375 66.025)
     (stroke (width 0.1) (type solid)) (layer "Edge.Cuts"))
-  (gr_line (start 161.798 59.53125) (end 157.956267 59.53125)
+  (gr_line (start 161.528125 59.53125) (end 157.956267 59.53125)
     (stroke (width 0.1) (type solid)) (layer "Edge.Cuts"))
   (gr_arc (start 95.39375 47.475) (mid 95.540197 47.121447) (end 95.89375 46.975)
@@
   (gr_line (start 128.44375 47.475) (end 128.44375 60.475)
     (stroke (width 0.1) (type solid)) (layer "Edge.Cuts"))
-  (gr_arc (start 161.798 48.41875) (mid 162.920478 48.883771) (end 163.3855 50.00625)
+  (gr_arc (start 161.528325 48.41875) (mid 162.650781 48.88378) (end 163.115825 50.00625)
     (stroke (width 0.1) (type solid)) (layer "Edge.Cuts"))
   (gr_arc (start 128.44375 60.475) (mid 128.297303 60.828553) (end 127.94375 60.975)
@@
   (gr_arc (start 108.89375 27.925) (mid 109.247303 28.071447) (end 109.39375 28.425)
     (stroke (width 0.1) (type solid)) (layer "Edge.Cuts"))
-  (gr_line (start 163.3855 50.00625) (end 163.3855 57.94375)
+  (gr_line (start 163.115725 50.00625) (end 163.115725 57.94375)
     (stroke (width 0.1) (type solid)) (layer "Edge.Cuts"))
   (gr_arc (start 147.49375 41.425) (mid 147.347303 41.778553) (end 146.99375 41.925)
@@
   (gr_line (start 109.39375 28.425) (end 109.39375 41.425)
     (stroke (width 0.1) (type solid)) (layer "Edge.Cuts"))
-  (gr_arc (start 163.3855 57.94375) (mid 162.920502 59.066253) (end 161.798 59.53125)
+  (gr_arc (start 163.115775 57.94375) (mid 162.650745 59.066256) (end 161.528225 59.53125)
     (stroke (width 0.1) (type solid)) (layer "Edge.Cuts"))
   (gr_arc (start 147.49375 60.475) (mid 147.347303 60.828553) (end 146.99375 60.975)
