File: KiCad/jam-pad-plate/jam-pad_plate.kicad_pcb (KiCad board)
At the start: 2 copper layers, 137.3 x 71.4 mm, 8 parts, among them SW14 RotaryEncoder_Switch

Commit message: fab, clover logo, some other stuff? idr sorry
Parts:
- removed SW14: RotaryEncoder_Switch, Keebio-Parts:RotaryEncoder_Alps_EC11E-Switch_Vertical_H20mm
Other:
- board size 137.3 x 71.4 mm -> 130.6 x 71.4 mm
- board text added: "JLCJLCJLCJLC"
